Commit message: Update robot.xacro

File: urdf/robot.xacro (robot description, xacro)
@@ -14,5 +14,5 @@
   </link>
   <joint name="base_link_joint" type="fixed">
-    <origin xyz="0 0 0" rpy="0 0 0" />
+    <origin xyz="0 0 0" rpy="0 0 -1.5707" />
     <parent link="base_footprint"/>
     <child link="chassis" />
